File: Eagle/tlc5916-2seg.sch (EAGLE design)
At the start: 8 parts, among them IC1 HD-A544D, U1 TLC5916IN, U2 TLC5916IN

Commit message: Updted R1, R2 to 1K (from 5K), added schematics Frame
Parts:
- R1, R2: value 5k -> 1k
Other:
- moved on the sheet: C1, C2, IC1, R1, R2, U1, U2, X1-1, X1-2, X1-3, X1-4, X1-5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
